Commit message: mando with more features

File: mando_description/urdf/mando.xacro (robot description, xacro)
@@ -1,4 +1,5 @@
 <?xml version="1.0"?>
 <robot name="mando" xmlns:xacro="http://www.ros.org/wiki/xacro">
+<xacro:include filename="$(find mando_description)/urdf/mando_gazebo.xacro" />
   <!-- Materials -->
   <material name="Black">
@@ -17,4 +18,5 @@
   <xacro:property name="baselink_height" value="0.35" />
   <xacro:property name="ground_clearance" value="0.15" />
+  <xacro:property name="castor_box" value="0.1"/>
   <!-- Base Footprint -->
   <link name="base_footprint">
@@ -23,6 +25,6 @@
   <link name="base_link">
   <inertial>
-    <mass value="30" />
-    <origin xyz="0 0 0" />
+    <mass value="400" />
+    <origin xyz="0 0 0" rpy="0 0 0"/>
     <inertia ixx="33.79" ixy="-0.03" ixz="2.67" iyy="53.15" iyz="0" izz="44.73" />
   </inertial>
@@ -34,4 +36,10 @@
     <material name="Red" />
   </visual>
+  <collision>
+    <origin rpy="0 0 0" xyz="0 -0.83 0.15" />
+    <geometry>
+      <mesh filename="package://mando_description/meshes/mando_chasis.STL" scale="0.001 0.001 0.001" />
+    </geometry>
+  </collision>
   </link>
   <joint name="basefootprint_to_baselink" type="fixed">
@@ -40,3 +48,287 @@
     <origin xyz="0 0 ${baselink_height+ground_clearance}" rpy="0 0 0" />
   </joint>
-</robot>
+  <!-- Castor Wheel Link-->
+  <link name="castor_wheel_box">
+    <inertial>
+      <mass value="5" />
+      <origin xzy="0 0 0" rpy="0 0 0" />
+      <!-- Taking inertia to be random values-->
+      <inertia ixx="0.1" ixy="0.1" ixz="0.1" iyy="0.1" iyz="0.1" izz="0.1" />
+    </inertial>
+    <visual>
+      <origin xyz="0 0 0" rpy="0 0 0" />
+      <geometry>
+        <box size="${castor_box} ${castor_box} ${castor_box}" />
+      </geometry>
+      <material name="Black" />
+    </visual>
+    <collision>
+      <origin xyz="0 0 0" rpy="0 0 0" />
+      <geometry>
+        <box size="${castor_box} ${castor_box} ${castor_box}" />
+      </geometry>
+    </collision>
+  </link>
+  <joint name="baselink_to_caster_wheel_box" type="continuous">
+    <parent link="base_link" />
+    <child link="castor_wheel_box" />
+    <origin xyz="-0.4 -0.03 -${baselink_height+0.05}" rpy="0 0 0" />
+    <axis xyz="0 0 1" rpy="0 0 0" />
+  </joint>
+  <!-- Castor Wheel Back Cylinder-->
+  <link name="castor_cylinder">
+    <inertial>
+      <mass value="5" />
+      <origin xyz="0 0 0" rpy="0 0 0" />
+      <!-- Taking inertia to be random values-->
+      <inertia ixx="0.1" ixy="0.1" ixz="0.1" iyy="0.1" iyz="0.1" izz="0.1" />
+    </inertial>
+    <visual>
+      <origin xyz="0 0 0" rpy="1.57 0 0" />
+      <geometry>
+        <cylinder radius="${(ground_clearance - castor_box/2)/2}" length="0.02" />
+      </geometry>
+      <material name="White" />
+    </visual>
+    <collision>
+      <origin xyz="0 0 0" rpy="1.57 0 0" />
+      <geometry>
+        <cylinder radius="${(ground_clearance - castor_box/2)/2}" length="0.02" />
+      </geometry>
+    </collision>
+  </link>
+  <joint name="castorwheel_to_castorbox" type="continuous">
+    <parent link="castor_wheel_box" />
+    <child link="castor_cylinder" />
+    <origin xyz="0 0 -${castor_box/2 - 0.02}" rpy="0 0 0" />
+    <axis xyz="0 1 0" rpy="0 0 0" />
+  </joint>
+  <!-- Castor Wheel Front Link-->
+  <link name="castor_wheel_box_front">
+    <inertial>
+      <mass value="5" />
+      <origin xzy="0 0 0" rpy="0 0 0" />
+      <!-- Taking inertia to be random values-->
+      <inertia ixx="0.1" ixy="0.1" ixz="0.1" iyy="0.1" iyz="0.1" izz="0.1" />
+    </inertial>
+    <visual>
+      <origin xyz="0 0 0" rpy="0 0 0" />
+      <geometry>
+        <box size="${castor_box} ${castor_box} ${castor_box}" />
+      </geometry>
+      <material name="Black" />
+    </visual>
+    <collision>
+      <origin xyz="0 0 0" rpy="0 0 0" />
+      <geometry>
+        <box size="${castor_box} ${castor_box} ${castor_box}" />
+      </geometry>
+    </collision>
+  </link>
+  <joint name="baselink_to_caster_wheel_box_front" type="continuous">
+    <parent link="base_link" />
+    <child link="castor_wheel_box_front" />
+    <origin xyz="0.45 -0.03 -${baselink_height+0.05}" rpy="0 0 0" />
+    <axis xyz="0 0 1" rpy="0 0 0" />
+  </joint>
+   <!-- Castor Wheel Front Cylinder-->
+  <link name="castor_cylinder_front">
+    <inertial>
+      <mass value="5" />
+      <origin xyz="0 0 0" rpy="0 0 0" />
+      <!-- Taking inertia to be random values-->
+      <inertia ixx="0.1" ixy="0.1" ixz="0.1" iyy="0.1" iyz="0.1" izz="0.1" />
+    </inertial>
+    <visual>
+      <origin xyz="0 0 0" rpy="1.57 0 0" />
+      <geometry>
+        <cylinder radius="${(ground_clearance - castor_box/2)/2}" length="0.02" />
+      </geometry>
+      <material name="White" />
+    </visual>
+    <collision>
+      <origin xyz="0 0 0" rpy="1.57 0 0" />
+      <geometry>
+        <cylinder radius="${(ground_clearance - castor_box/2)/2}" length="0.02" />
+      </geometry>
+    </collision>
+  </link>
+  <joint name="castorwheelfront_to_castorbox" type="continuous">
+    <parent link="castor_wheel_box_front" />
+    <child link="castor_cylinder_front" />
+    <origin xyz="0 0 -${castor_box/2 - 0.02}" rpy="0 0 0" />
+    <axis xyz="0 1 0" rpy="0 0 0" />
+  </joint>
+ <!--Left Wheel for Bot-->
+  <link name="left_wheel">
+    <inertial>
+      <mass value="5" />
+      <origin xyz="0 0 0" rpy="0 0 0" />
+      <!-- Taking inertia to be random values-->
+      <inertia ixx="0.1" ixy="0.1" ixz="0.1" iyy="0.1" iyz="0.1" izz="0.1" />
+    </inertial>
+    <visual>
+    <origin rpy="0 0 0" xyz="0 0 0" />
+    <geometry>
+      <mesh filename="package://mando_description/meshes/wheel.dae" scale="0.83 0.83 0.83" />
+    </geometry>
+    </visual>
+    <collision>
+      <origin rpy="0 0 0" xyz="0 0 0" />
+      <geometry>
+        <mesh filename="package://mando_description/meshes/wheel.dae" scale="0.83 0.83 0.83" />
+      </geometry>
+    </collision>
+  </link>
+  <joint name="left_wheel_to_base_link" type="continuous" >
+    <parent link="base_link" />
+    <child link="left_wheel" />
+    <origin xyz="0.306 0.3302 -${baselink_height}" rpy="0 0 0" />
+    <axis xyz="0 2 0" rpy="0 0 0" />
+  </joint>
+  <transmission name="left_wheel_joint_trans">
+    <type>transmission_interface/SimpleTransmission</type>
+    <joint name="left_wheel_to_base_link"/>
+    <actuator name="left_wheel_joint_motor">
+      <hardwareInterface>EffortJointInterface</hardwareInterface>
+      <mechanicalReduction>1</mechanicalReduction>
+    </actuator>
+  </transmission>
+   <!--Right Wheel for Bot-->
+  <link name="right_wheel">
+    <inertial>
+      <mass value="5" />
+      <origin xyz="0 0 0" rpy="0 0 0" />
+      <!-- Taking inertia to be random values-->
+      <inertia ixx="0.1" ixy="0.1" ixz="0.1" iyy="0.1" iyz="0.1" izz="0.1" />
+    </inertial>
+    <visual>
+    <origin rpy="0 0 0" xyz="0 0 0" />
+    <geometry>
+      <mesh filename="package://mando_description/meshes/wheel.dae" scale="0.83 0.83 0.83" />
+    </geometry>
+    </visual>
+    <collision>
+      <origin rpy="0 0 0" xyz="0 0 0" />
+      <geometry>
+       <mesh filename="package://mando_description/meshes/wheel.dae" scale="0.83 0.83 0.83" />
+      </geometry>
+    </collision>
+  </link>
+  <joint name="right_wheel_to_base_link" type="continuous" >
+    <parent link="base_link" />
+    <child link="right_wheel" />
+    <origin xyz="0.306 -0.4 -${baselink_height}" rpy="0 0 0" />
+    <axis xyz="0 2 0" rpy="0 0 0" />
+  </joint>
+  <transmission name="right_wheel_joint_trans">
+    <type>transmission_interface/SimpleTransmission</type>
+    <joint name="right_wheel_to_base_link"/>
+    <actuator name="right_wheel_joint_motor">
+      <hardwareInterface>EffortJointInterface</hardwareInterface>
+      <mechanicalReduction>1</mechanicalReduction>
+    </actuator>
+  </transmission>
+    <!-- Camera link-->
+  <link name="camera">
+    <inertial>
+      <mass value="3" />
+      <origin xyz="0 0 0" rpy="0 0 0" />
+      <!-- Taking inertia to be random values-->
+      <inertia ixx="0.1" ixy="0.1" ixz="0.1" iyy="0.1" iyz="0.1" izz="0.1" />
+    </inertial>
+    <visual>
+    <origin rpy="0 0 0" xyz="0 0 0" />
+    <geometry>
+        <box size="0.05 0.05 0.05" />
+    </geometry>
+    <material name="Black" />
+    </visual>
+    <collision>
+      <origin rpy="0 0 0" xyz="0 0 0" />
+      <geometry>
+        <box size="0.05 0.05 0.05" />
+      </geometry>
+    </collision>
+  </link>
+  <joint name="base_link_to_camera" type="fixed">
+    <parent link="base_link" />
+    <child link="camera" />
+    <origin xyz="0.17 -0.03 1.292471" rpy="0 0 0" />
+  </joint>
+  <!-- Lidar Link-->
+  <link name="Lidar">
+    <inertial>
+      <mass value="3" />
+      <origin xyz="0 0 0" rpy="0 0 0" />
+      <!-- Taking inertia to be random values-->
+      <inertia ixx="0.1" ixy="0.1" ixz="0.1" iyy="0.1" iyz="0.1" izz="0.1" />
+    </inertial>
+    <visual>
+      <origin xyz="0 0 0" rpy="0 0 0" />
+      <geometry>
+        <mesh filename="package://mando_description/meshes/lidar.stl" scale="0.001 0.001 0.001" />
+      </geometry>
+      <material name="White" />
+    </visual>
+    <collision>
+      <origin xyz="0 0 0" rpy="0 0 0" />
+      <geometry>
+        <mesh filename="package://mando_description/meshes/lidar.stl" scale="0.001 0.001 0.001" />
+      </geometry>
+    </collision>
+  </link>
+  <joint name="base_link_to_lidar" type="fixed">
+    <parent link="base_link" />
+    <child link="Lidar" />
+    <origin xyz="0.6 0 -0.175423" rpy="0 0 -1.57" />
+  </joint>
+  <!-- IMU link-->
+  <link name="IMU">
+    <inertial>
+      <mass value="3" />
+      <origin xyz="0 0 0" rpy="0 0 0" />
+      <!-- Taking inertia to be random values-->
+      <inertia ixx="0.1" ixy="0.1" ixz="0.1" iyy="0.1" iyz="0.1" izz="0.1" />
+    </inertial>
+    <visual>
+    <origin xyz="0 0 0" rpy="0 0 0" />
+    <geometry>
+      <box size="0.05 0.05 0.05" />
+    </geometry>
+    </visual>
+    <collision>
+      <origin xyz="0 0 0" rpy="0 0 0" />
+      <geometry>
+        <box size="0.05 0.05 0.05" />
+      </geometry>
+    </collision>
+  </link>
+  <joint name="base_link_to_IMU" type="fixed">
+    <parent link="base_link" />
+    <child link="IMU"/>
+    <origin xyz="0.325775 -0.03 0.198187" rpy="0 0 0"/>
+  </joint>
+  <!-- Plugin for differential drive -->
+	<gazebo>
+    <plugin filename="libgazebo_ros_diff_drive.so" name="differential_drive_controller">
+      <rosDebugLevel>Debug</rosDebugLevel>
+      <publishWheelTF>True</publishWheelTF>
+      <publishTf>1</publishTf>
+      <publishWheelJointState>true</publishWheelJointState>
+      <alwaysOn>true</alwaysOn>
+      <updateRate>20</updateRate>
+      <leftJoint>left_wheel_to_base_link</leftJoint>
+      <rightJoint>right_wheel_to_base_link</rightJoint>
+      <wheelSeparation>0.622308</wheelSeparation>
+      <wheelDiameter>0.2808</wheelDiameter>
+      <broadcastTF>1</broadcastTF>
+      <wheelTorque>1000</wheelTorque>
+      <wheelAcceleration>200</wheelAcceleration>
+      <commandTopic>cmd_vel</commandTopic>
+      <odometryFrame>odom</odometryFrame>
+      <odometryTopic>odom</odometryTopic>
+      <robotBaseFrame>base_footprint</robotBaseFrame>
+    </plugin>
+  </gazebo>
+ </robot>
