Commit message: added all sensors to urdf and new urdf

File: mando_description/urdf/mando.xacro (robot description, xacro)
@@ -1,316 +1,313 @@
 <?xml version="1.0"?>
-<robot name="mando" xmlns:xacro="http://www.ros.org/wiki/xacro">
-<xacro:include filename="$(find mando_description)/urdf/mando_gazebo.xacro" />
-  <!-- Materials -->
+<robot name="mando"
+  xmlns:xacro="http://www.ros.org/wiki/xacro">
+  <!-- Defining the colors used in this robot -->
   <material name="Black">
-    <color rgba="0.0 0.0 0.0 1.0" />
+    <color rgba="0.0 0.0 0.0 1.0"/>
   </material>
   <material name="Red">
-    <color rgba="0.8 0.0 0.0 1.0" />
+    <color rgba="0.8 0.0 0.0 1.0"/>
   </material>
   <material name="White">
-    <color rgba="1.0 1.0 1.0 1.0" />
+    <color rgba="1.0 1.0 1.0 1.0"/>
   </material>
   <material name="Blue">
-    <color rgba="0.0 0.0 0.8 1.0" />
+    <color rgba="0.0 0.0 0.8 1.0"/>
   </material>
-  <!-- Xacro Properties -->
-  <xacro:property name="baselink_height" value="0.35" />
-  <xacro:property name="ground_clearance" value="0.15" />
-  <xacro:property name="castor_box" value="0.1"/>
-  <!-- Base Footprint -->
+  <!-- PROPERTY LIST -->
+  <!--All units in m-kg-s-radians unit system -->
+  <!-- Main body radius and height -->
+  <!-- Main Body Cylinder base   -->
+  <!-- in kg-->
+  <!-- caster wheel radius and height -->
+  <!-- caster wheel mass -->
+  <!-- in kg-->
+  <!-- caster wheel radius and height -->
+  <!-- caster wheel mass -->
+  <!-- in kg-->
+  <!-- Wheels -->
+  <!-- in kg-->
+  <!-- Hokuyo Laser scanner -->
+  <!-- Macro for calculating inertia of cylinder -->
+  <!-- BASE-FOOTPRINT -->
+  <!-- base_footprint is a fictitious link(frame) that is on the ground right below base_link origin -->
   <link name="base_footprint">
-  </link>
-  <!-- Baselink -->
+    <inertial>
+      <mass value="0.0001"/>
+      <origin xyz="0 0 0"/>
+      <inertia ixx="0.0001" ixy="0.0" ixz="0.0" iyy="0.0001" iyz="0.0" izz="0.0001"/>
+    </inertial>
+    <visual>
+      <origin rpy="0 0 0" xyz="0 0 0"/>
+      <geometry>
+        <box size="0.001 0.001 0.001"/>
+      </geometry>
+    </visual>
+  </link>
+  <joint name="base_footprint_joint" type="fixed">
+    <origin rpy="0 0 0" xyz="0 0 0.04"/>
+    <parent link="base_footprint"/>
+    <child link="base_link"/>
+  </joint>
+  <!-- BASE-LINK -->
+  <!--Actual body/chassis of the robot-->
   <link name="base_link">
-  <inertial>
-    <mass value="400" />
-    <origin xyz="0 0 0" rpy="0 0 0"/>
-    <inertia ixx="33.79" ixy="-0.03" ixz="2.67" iyy="53.15" iyz="0" izz="44.73" />
-  </inertial>
-  <visual>
-    <origin rpy="0 0 0" xyz="0 -0.83 0.15" />
-    <geometry>
-      <mesh filename="package://mando_description/meshes/mando_chasis.STL" scale="0.001 0.001 0.001" />
-    </geometry>
-    <material name="Red" />
-  </visual>
-  <collision>
-    <origin rpy="0 0 0" xyz="0 -0.83 0.15" />
-    <geometry>
-      <mesh filename="package://mando_description/meshes/mando_chasis.STL" scale="0.001 0.001 0.001" />
-    </geometry>
-  </collision>
-  </link>
-  <joint name="basefootprint_to_baselink" type="fixed">
-    <parent link="base_footprint" />
-    <child link="base_link" />
-    <origin xyz="0 0 ${baselink_height+ground_clearance}" rpy="0 0 0" />
-  </joint>
-  <!-- Castor Wheel Link-->
-  <link name="castor_wheel_box">
-    <inertial>
-      <mass value="5" />
-      <origin xzy="0 0 0" rpy="0 0 0" />
-      <!-- Taking inertia to be random values-->
-      <inertia ixx="0.1" ixy="0.1" ixz="0.1" iyy="0.1" iyz="0.1" izz="0.1" />
-    </inertial>
-    <visual>
-      <origin xyz="0 0 0" rpy="0 0 0" />
-      <geometry>
-        <box size="${castor_box} ${castor_box} ${castor_box}" />
-      </geometry>
-      <material name="Black" />
+    <inertial>
+      <mass value="5"/>
+      <origin xyz="0 0 0"/>
+      <!--The 3x3 rotational inertia matrix. -->
+      <inertia ixx="0.0282916666667" ixy="0" ixz="0" iyy="0.0282916666667" iyz="0" izz="0.05625"/>
+    </inertial>
+    <visual>
+      <origin rpy="0 0 0" xyz="0 0 0"/>
+      <geometry>
+        <cylinder length="0.02" radius="0.15"/>
+      </geometry>
+      <material name="White"/>
     </visual>
     <collision>
-      <origin xyz="0 0 0" rpy="0 0 0" />
-      <geometry>
-        <box size="${castor_box} ${castor_box} ${castor_box}" />
+      <origin rpy="0 0 0 " xyz="0 0 0"/>
+      <geometry>
+        <cylinder length="0.02" radius="0.15"/>
       </geometry>
     </collision>
   </link>
-  <joint name="baselink_to_caster_wheel_box" type="continuous">
-    <parent link="base_link" />
-    <child link="castor_wheel_box" />
-    <origin xyz="-0.4 -0.03 -${baselink_height+0.05}" rpy="0 0 0" />
-    <axis xyz="0 0 1" rpy="0 0 0" />
-  </joint>
-  <!-- Castor Wheel Back Cylinder-->
-  <link name="castor_cylinder">
-    <inertial>
-      <mass value="5" />
-      <origin xyz="0 0 0" rpy="0 0 0" />
-      <!-- Taking inertia to be random values-->
-      <inertia ixx="0.1" ixy="0.1" ixz="0.1" iyy="0.1" iyz="0.1" izz="0.1" />
-    </inertial>
-    <visual>
-      <origin xyz="0 0 0" rpy="1.57 0 0" />
-      <geometry>
-        <cylinder radius="${(ground_clearance - castor_box/2)/2}" length="0.02" />
-      </geometry>
-      <material name="White" />
+  <!--fb : front, back ; lr: left, right -->
+  <link name="front_right_wheel">
+    <visual>
+      <origin rpy="1.57079632679 0  0 " xyz="0 0 0"/>
+      <geometry>
+        <cylinder length="0.02" radius="0.04"/>
+      </geometry>
+      <material name="DarkGray"/>
     </visual>
     <collision>
-      <origin xyz="0 0 0" rpy="1.57 0 0" />
-      <geometry>
-        <cylinder radius="${(ground_clearance - castor_box/2)/2}" length="0.02" />
+      <origin rpy="1.57079632679 0 0 " xyz="0 0 0"/>
+      <geometry>
+        <cylinder length="0.02" radius="0.04"/>
       </geometry>
     </collision>
-  </link>
-  <joint name="castorwheel_to_castorbox" type="continuous">
-    <parent link="castor_wheel_box" />
-    <child link="castor_cylinder" />
-    <origin xyz="0 0 -${castor_box/2 - 0.02}" rpy="0 0 0" />
-    <axis xyz="0 1 0" rpy="0 0 0" />
-  </joint>
-  <!-- Castor Wheel Front Link-->
-  <link name="castor_wheel_box_front">
-    <inertial>
-      <mass value="5" />
-      <origin xzy="0 0 0" rpy="0 0 0" />
-      <!-- Taking inertia to be random values-->
-      <inertia ixx="0.1" ixy="0.1" ixz="0.1" iyy="0.1" iyz="0.1" izz="0.1" />
-    </inertial>
-    <visual>
-      <origin xyz="0 0 0" rpy="0 0 0" />
-      <geometry>
-        <box size="${castor_box} ${castor_box} ${castor_box}" />
-      </geometry>
-      <material name="Black" />
-    </visual>
-    <collision>
-      <origin xyz="0 0 0" rpy="0 0 0" />
-      <geometry>
-        <box size="${castor_box} ${castor_box} ${castor_box}" />
-      </geometry>
-    </collision>
-  </link>
-  <joint name="baselink_to_caster_wheel_box_front" type="continuous">
-    <parent link="base_link" />
-    <child link="castor_wheel_box_front" />
-    <origin xyz="0.45 -0.03 -${baselink_height+0.05}" rpy="0 0 0" />
-    <axis xyz="0 0 1" rpy="0 0 0" />
-  </joint>
-   <!-- Castor Wheel Front Cylinder-->
-  <link name="castor_cylinder_front">
-    <inertial>
-      <mass value="5" />
-      <origin xyz="0 0 0" rpy="0 0 0" />
-      <!-- Taking inertia to be random values-->
-      <inertia ixx="0.1" ixy="0.1" ixz="0.1" iyy="0.1" iyz="0.1" izz="0.1" />
-    </inertial>
-    <visual>
-      <origin xyz="0 0 0" rpy="1.57 0 0" />
-      <geometry>
-        <cylinder radius="${(ground_clearance - castor_box/2)/2}" length="0.02" />
-      </geometry>
-      <material name="White" />
-    </visual>
-    <collision>
-      <origin xyz="0 0 0" rpy="1.57 0 0" />
-      <geometry>
-        <cylinder radius="${(ground_clearance - castor_box/2)/2}" length="0.02" />
-      </geometry>
-    </collision>
-  </link>
-  <joint name="castorwheelfront_to_castorbox" type="continuous">
-    <parent link="castor_wheel_box_front" />
-    <child link="castor_cylinder_front" />
-    <origin xyz="0 0 -${castor_box/2 - 0.02}" rpy="0 0 0" />
-    <axis xyz="0 1 0" rpy="0 0 0" />
-  </joint>
- <!--Left Wheel for Bot-->
-  <link name="left_wheel">
-    <inertial>
-      <mass value="5" />
-      <origin xyz="0 0 0" rpy="0 0 0" />
-      <!-- Taking inertia to be random values-->
-      <inertia ixx="0.1" ixy="0.1" ixz="0.1" iyy="0.1" iyz="0.1" izz="0.1" />
-    </inertial>
-    <visual>
-    <origin rpy="0 0 0" xyz="0 0 0" />
-    <geometry>
-      <mesh filename="package://mando_description/meshes/wheel.dae" scale="0.83 0.83 0.83" />
-    </geometry>
-    </visual>
-    <collision>
-      <origin rpy="0 0 0" xyz="0 0 0" />
-      <geometry>
-        <mesh filename="package://mando_description/meshes/wheel.dae" scale="0.83 0.83 0.83" />
-      </geometry>
-    </collision>
-  </link>
-  <joint name="left_wheel_to_base_link" type="continuous" >
-    <parent link="base_link" />
-    <child link="left_wheel" />
-    <origin xyz="0.306 0.3302 -${baselink_height}" rpy="0 0 0" />
-    <axis xyz="0 2 0" rpy="0 0 0" />
-  </joint>
-  <transmission name="left_wheel_joint_trans">
+    <inertial>
+      <mass value="2.5"/>
+      <origin xyz="0 0 0"/>
+      <inertia ixx="0.00108333333333" ixy="0" ixz="0" iyy="0.00108333333333" iyz="0" izz="0.002"/>
+    </inertial>
+  </link>
+  <joint name="front_right_wheel_joint" type="continuous">
+    <parent link="base_link"/>
+    <child link="front_right_wheel"/>
+    <origin rpy="0 0 0" xyz="0.0 0.15 0.0"/>
+    <axis rpy="0  0" xyz="0 1 0"/>
+    <limit effort="100" velocity="100"/>
+    <joint_properties damping="0.0" friction="0.0"/>
+  </joint>
+  <!-- Transmission is important to link the joints and the controller -->
+  <transmission name="front_right_wheel_joint_trans">
     <type>transmission_interface/SimpleTransmission</type>
-    <joint name="left_wheel_to_base_link"/>
-    <actuator name="left_wheel_joint_motor">
+    <joint name="front_right_wheel_joint"/>
+    <actuator name="front_right_wheel_joint_motor">
       <hardwareInterface>EffortJointInterface</hardwareInterface>
       <mechanicalReduction>1</mechanicalReduction>
     </actuator>
   </transmission>
-   <!--Right Wheel for Bot-->
-  <link name="right_wheel">
-    <inertial>
-      <mass value="5" />
-      <origin xyz="0 0 0" rpy="0 0 0" />
-      <!-- Taking inertia to be random values-->
-      <inertia ixx="0.1" ixy="0.1" ixz="0.1" iyy="0.1" iyz="0.1" izz="0.1" />
-    </inertial>
-    <visual>
-    <origin rpy="0 0 0" xyz="0 0 0" />
-    <geometry>
-      <mesh filename="package://mando_description/meshes/wheel.dae" scale="0.83 0.83 0.83" />
-    </geometry>
+  <!--fb : front, back ; lr: left, right -->
+  <link name="front_left_wheel">
+    <visual>
+      <origin rpy="1.57079632679 0  0 " xyz="0 0 0"/>
+      <geometry>
+        <cylinder length="0.02" radius="0.04"/>
+      </geometry>
+      <material name="DarkGray"/>
     </visual>
     <collision>
-      <origin rpy="0 0 0" xyz="0 0 0" />
-      <geometry>
-       <mesh filename="package://mando_description/meshes/wheel.dae" scale="0.83 0.83 0.83" />
+      <origin rpy="1.57079632679 0 0 " xyz="0 0 0"/>
+      <geometry>
+        <cylinder length="0.02" radius="0.04"/>
       </geometry>
     </collision>
-  </link>
-  <joint name="right_wheel_to_base_link" type="continuous" >
-    <parent link="base_link" />
-    <child link="right_wheel" />
-    <origin xyz="0.306 -0.4 -${baselink_height}" rpy="0 0 0" />
-    <axis xyz="0 2 0" rpy="0 0 0" />
-  </joint>
-  <transmission name="right_wheel_joint_trans">
+    <inertial>
+      <mass value="2.5"/>
+      <origin xyz="0 0 0"/>
+      <inertia ixx="0.00108333333333" ixy="0" ixz="0" iyy="0.00108333333333" iyz="0" izz="0.002"/>
+    </inertial>
+  </link>
+  <joint name="front_left_wheel_joint" type="continuous">
+    <parent link="base_link"/>
+    <child link="front_left_wheel"/>
+    <origin rpy="0 0 0" xyz="0.0 -0.15 0.0"/>
+    <axis rpy="0  0" xyz="0 1 0"/>
+    <limit effort="100" velocity="100"/>
+    <joint_properties damping="0.0" friction="0.0"/>
+  </joint>
+  <!-- Transmission is important to link the joints and the controller -->
+  <transmission name="front_left_wheel_joint_trans">
     <type>transmission_interface/SimpleTransmission</type>
-    <joint name="right_wheel_to_base_link"/>
-    <actuator name="right_wheel_joint_motor">
+    <joint name="front_left_wheel_joint"/>
+    <actuator name="front_left_wheel_joint_motor">
       <hardwareInterface>EffortJointInterface</hardwareInterface>
       <mechanicalReduction>1</mechanicalReduction>
     </actuator>
   </transmission>
-    <!-- Camera link-->
-  <link name="camera">
-    <inertial>
-      <mass value="3" />
-      <origin xyz="0 0 0" rpy="0 0 0" />
-      <!-- Taking inertia to be random values-->
-      <inertia ixx="0.1" ixy="0.1" ixz="0.1" iyy="0.1" iyz="0.1" izz="0.1" />
-    </inertial>
-    <visual>
-    <origin rpy="0 0 0" xyz="0 0 0" />
-    <geometry>
-        <box size="0.05 0.05 0.05" />
-    </geometry>
-    <material name="Black" />
+  <!--Caster front  -->
+  <link name="caster_front_link">
+    <visual>
+      <origin rpy="1.57079632679 0 0" xyz="0 0.02 0"/>
+      <geometry>
+        <sphere radius="0.025"/>
+      </geometry>
+      <material name="Black"/>
     </visual>
     <collision>
-      <origin rpy="0 0 0" xyz="0 0 0" />
-      <geometry>
-        <box size="0.05 0.05 0.05" />
-      </geometry>
+      <geometry>
+        <sphere radius="0.025"/>
+      </geometry>
+      <origin rpy="1.57079632679 0 0" xyz="0 0.02 0"/>
     </collision>
-  </link>
-  <joint name="base_link_to_camera" type="fixed">
-    <parent link="base_link" />
-    <child link="camera" />
-    <origin xyz="0.17 -0.03 1.292471" rpy="0 0 0" />
-  </joint>
-  <!-- Lidar Link-->
-  <link name="Lidar">
-    <inertial>
-      <mass value="3" />
-      <origin xyz="0 0 0" rpy="0 0 0" />
-      <!-- Taking inertia to be random values-->
-      <inertia ixx="0.1" ixy="0.1" ixz="0.1" iyy="0.1" iyz="0.1" izz="0.1" />
-    </inertial>
-    <visual>
-      <origin xyz="0 0 0" rpy="0 0 0" />
-      <geometry>
-        <mesh filename="package://mando_description/meshes/lidar.stl" scale="0.001 0.001 0.001" />
-      </geometry>
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