Commit message: fixed default param warnings

File: kbot/urdf/kbot.xacro (robot description, xacro)
@@ -1,20 +1,20 @@
-<?xml version="1.0"?>
-<robot name= "mando">
+<?xml version="1.0" ?>
+<robot name="mando">
   <link name="base_link">
     <inertial>
-      <mass value="1.0"/>
-      <inertia ixx="0.015" iyy="0.0375" izz="0.0375" ixy="0" ixz="0" iyz="0"/>
-    </inertial>
-    <visual>
-      <geometry>
-        <box size="1.16195 0.651 0.77596"/>
+      <mass value="1.0" />
+      <inertia ixx="0.015" iyy="0.0375" izz="0.0375" ixy="0" ixz="0" iyz="0" />
+    </inertial>
+    <visual>
+      <geometry>
+        <box size="1.16195 0.651 0.77596" />
       </geometry>
       <material name="silver">
-        <color rgba="0.75 0.75 0.75 1"/>
+        <color rgba="0.75 0.75 0.75 1" />
       </material>
     </visual>
     <collision>
       <geometry>
-        <box size="0.6 0.3 0.3"/>
+        <box size="0.6 0.3 0.3" />
       </geometry>
     </collision>
@@ -22,211 +22,221 @@
   <link name="back_caster">
     <inertial>
-      <mass value="0.1"/>
-      <inertia ixx="0.00083" iyy="0.00083" izz="0.000167" ixy="0" ixz="0" iyz="0"/>
-    </inertial>
-    <visual>
-      <geometry>
-        <box size="0.1 0.1 0.77596"/>
-      </geometry>
-      <material name="silver"/>
-    </visual>
-    <collision>
-      <geometry>
-        <box size="0.1 0.1 0.77596"/>
+      <mass value="0.1" />
+      <inertia ixx="0.00083" iyy="0.00083" izz="0.000167" ixy="0" ixz="0" iyz="0" />
+    </inertial>
+    <visual>
+      <geometry>
+        <box size="0.1 0.1 0.77596" />
+      </geometry>
+      <material name="silver" />
+    </visual>
+    <collision>
+      <geometry>
+        <box size="0.1 0.1 0.77596" />
       </geometry>
     </collision>
   </link>
   <joint name="back_caster_joint" type="continuous">
-    <axis xyz="0 0 1"/>
-    <parent link="base_link"/>
-    <child link="back_caster"/>
-    <origin rpy="0 0 0" xyz="-0.491695 0 0"/>
+    <axis xyz="0 0 1" />
+    <parent link="base_link" />
+    <child link="back_caster" />
+    <origin rpy="0 0 0" xyz="-0.491695 0 0" />
   </joint>
   <link name="back_wheel">
     <inertial>
-      <mass value="0.1"/>
-      <inertia ixx="5.1458e-5" iyy="5.1458e-5" izz="6.125e-5" ixy="0" ixz="0" iyz="0"/>
-    </inertial>
-    <visual>
-      <geometry>
-        <cylinder length="0.05" radius="0.1"/>
-      </geometry>
-      <material name="black"/>
-    </visual>
-    <collision>
-      <geometry>
-        <cylinder length="0.05" radius="0.1"/>
+      <mass value="0.1" />
+      <inertia ixx="5.1458e-5" iyy="5.1458e-5" izz="6.125e-5" ixy="0" ixz="0" iyz="0" />
+    </inertial>
+    <visual>
+      <geometry>
+        <cylinder length="0.05" radius="0.1" />
+      </geometry>
+      <material name="black" />
+    </visual>
+    <collision>
+      <geometry>
+        <cylinder length="0.05" radius="0.1" />
       </geometry>
     </collision>
   </link>
   <joint name="back_wheel_joint" type="continuous">
-    <axis xyz="0 0 1"/>
-    <parent link="back_caster"/>
-    <child link="back_wheel"/>
-    <origin rpy="-1.5708 0 0" xyz="0.05 0 -.38798"/>
+    <axis xyz="0 0 1" />
+    <parent link="back_caster" />
+    <child link="back_wheel" />
+    <origin rpy="-1.5708 0 0" xyz="0.05 0 -.38798" />
   </joint>
   <link name="front_caster">
     <inertial>
-      <mass value="0.1"/>
-      <inertia ixx="0.00083" iyy="0.00083" izz="0.000167" ixy="0" ixz="0" iyz="0"/>
-    </inertial>
-    <visual>
-      <geometry>
-        <box size="0.1 0.1 0.77596"/>
-      </geometry>
-      <material name="silver"/>
-    </visual>
-    <collision>
-      <geometry>
-        <box size="0.1 0.1 0.77596"/>
+      <mass value="0.1" />
+      <inertia ixx="0.00083" iyy="0.00083" izz="0.000167" ixy="0" ixz="0" iyz="0" />
+    </inertial>
+    <visual>
+      <geometry>
+        <box size="0.1 0.1 0.77596" />
+      </geometry>
+      <material name="silver" />
+    </visual>
+    <collision>
+      <geometry>
+        <box size="0.1 0.1 0.77596" />
       </geometry>
     </collision>
   </link>
   <joint name="front_caster_joint" type="continuous">
-    <axis xyz="0 0 1"/>
-    <parent link="base_link"/>
-    <child link="front_caster"/>
-    <origin rpy="0 0 0" xyz="0.491695 0 0"/>
+    <axis xyz="0 0 1" />
+    <parent link="base_link" />
+    <child link="front_caster" />
+    <origin rpy="0 0 0" xyz="0.491695 0 0" />
   </joint>
   <link name="front_wheel">
     <inertial>
-      <mass value="0.1"/>
-      <inertia ixx="5.1458e-5" iyy="5.1458e-5" izz="6.125e-5" ixy="0" ixz="0" iyz="0"/>
-    </inertial>
-    <visual>
-      <geometry>
-        <cylinder length="0.05" radius="0.1"/>
-      </geometry>
-      <material name="black"/>
-    </visual>
-    <collision>
-      <geometry>
-        <cylinder length="0.05" radius="0.1"/>
+      <mass value="0.1" />
+      <inertia ixx="5.1458e-5" iyy="5.1458e-5" izz="6.125e-5" ixy="0" ixz="0" iyz="0" />
+    </inertial>
+    <visual>
+      <geometry>
+        <cylinder length="0.05" radius="0.1" />
+      </geometry>
+      <material name="black" />
+    </visual>
+    <collision>
+      <geometry>
+        <cylinder length="0.05" radius="0.1" />
       </geometry>
     </collision>
   </link>
   <joint name="front_wheel_joint" type="continuous">
-    <axis xyz="0 0 1"/>
-    <parent link="front_caster"/>
-    <child link="front_wheel"/>
-    <origin rpy="-1.5708 0 0" xyz="0.05 0 -.38798"/>
+    <axis xyz="0 0 1" />
+    <parent link="front_caster" />
+    <child link="front_wheel" />
+    <origin rpy="-1.5708 0 0" xyz="0.05 0 -.38798" />
   </joint>
   <link name="right_wheel">
     <inertial>
-      <mass value="0.1"/>
-      <inertia ixx="5.1458e-5" iyy="5.1458e-5" izz="6.125e-5" ixy="0" ixz="0" iyz="0"/>
-    </inertial>
-    <visual>
-      <geometry>
-        <cylinder length="0.05" radius="0.1"/>
+      <mass value="0.1" />
+      <inertia ixx="5.1458e-5" iyy="5.1458e-5" izz="6.125e-5" ixy="0" ixz="0" iyz="0" />
+    </inertial>
+    <visual>
+      <geometry>
+        <cylinder length="0.05" radius="0.1" />
       </geometry>
       <material name="black">
-        <color rgba="0 0 0 1"/>
+        <color rgba="0 0 0 1" />
       </material>
     </visual>
     <collision>
       <geometry>
-        <cylinder length="0.05" radius="0.1"/>
+        <cylinder length="0.05" radius="0.1" />
       </geometry>
     </collision>
   </link>
   <joint name="right_wheel_joint" type="continuous">
-    <axis xyz="0 0 1"/>
-    <parent link="base_link"/>
-    <child link="right_wheel"/>
-    <origin rpy="-1.5708 0 0" xyz="0.159795 -.3005 -.38798"/>
+    <axis xyz="0 0 1" />
+    <parent link="base_link" />
+    <child link="right_wheel" />
+    <origin rpy="-1.5708 0 0" xyz="0.159795 -.3005 -.38798" />
   </joint>
   <link name="left_wheel">
     <inertial>
-      <mass value="0.1"/>
-      <inertia ixx="5.1458e-5" iyy="5.1458e-5" izz="6.125e-5" ixy="0" ixz="0" iyz="0"/>
-    </inertial>
-    <visual>
-      <geometry>
-        <cylinder length="0.05" radius="0.1"/>
-      </geometry>
-      <material name="black"/>
-    </visual>
-    <collision>
-      <geometry>
-        <cylinder length="0.05" radius="0.1"/>
+      <mass value="0.1" />
+      <inertia ixx="5.1458e-5" iyy="5.1458e-5" izz="6.125e-5" ixy="0" ixz="0" iyz="0" />
+    </inertial>
+    <visual>
+      <geometry>
+        <cylinder length="0.05" radius="0.1" />
+      </geometry>
+      <material name="black" />
+    </visual>
+    <collision>
+      <geometry>
+        <cylinder length="0.05" radius="0.1" />
       </geometry>
     </collision>
   </link>
   <joint name="left_wheel_joint" type="continuous">
-    <axis xyz="0 0 1"/>
-    <parent link="base_link"/>
-    <child link="left_wheel"/>
-    <origin rpy="-1.5708 0 0" xyz="0.159795 0.3005 -.38978"/>
+    <axis xyz="0 0 1" />
+    <parent link="base_link" />
+    <child link="left_wheel" />
+    <origin rpy="-1.5708 0 0" xyz="0.159795 0.3005 -.38978" />
   </joint>
   <link name="hokuyo_link">
     <collision>
-      <origin xyz="0 0 0" rpy="0 0 0"/>
-      <geometry>
-        <box size="0.1 0.1 0.1"/>
-      </geometry>
-    </collision>
-    <visual>
-      <origin xyz="0 0 0" rpy="0 0 0"/>
-      <geometry>
-        <box size="0.1 0.1 0.1"/>
+      <origin xyz="0 0 0" rpy="0 0 0" />
+      <geometry>
+        <box size="0.1 0.1 0.1" />
+      </geometry>
+    </collision>
+    <visual>
+      <origin xyz="0 0 0" rpy="0 0 0" />
+      <geometry>
+        <box size="0.1 0.1 0.1" />
       </geometry>
     </visual>
     <inertial>
       <mass value="1e-5" />
-      <origin xyz="0 0 0" rpy="0 0 0"/>
+      <origin xyz="0 0 0" rpy="0 0 0" />
       <inertia ixx="1e-6" ixy="0" ixz="0" iyy="1e-6" iyz="0" izz="1e-6" />
     </inertial>
   </link>
   <joint name="hokuyo_joint" type="fixed">
-    <origin xyz="0.630975 0 -0.1807467" rpy="0 0 0"/>
-    <parent link="base_link"/>
-    <child link="hokuyo_link"/>
+    <origin xyz="0.630975 0 -0.1807467" rpy="0 0 0" />
+    <parent link="base_link" />
+    <child link="hokuyo_link" />
   </joint>
   <link name="camera_link">
     <visual>
-      <origin rpy="0 0 0" xyz="0 0 0"/>
-      <geometry>
-        <box size="0.05 0.05 0.05"/>
-      </geometry>
-      <material name="Blue"/>
+      <origin rpy="0 0 0" xyz="0 0 0" />
+      <geometry>
+        <box size="0.05 0.05 0.05" />
+      </geometry>
+      <material name="Blue" />
     </visual>
   </link>
   <joint name="camera_joint" type="fixed">
-    <origin rpy="0 1.0466 0" xyz="0.555975 0 0.72404"/>
-    <parent link="base_link"/>
-    <child link="camera_link"/>
+    <origin rpy="0 1.0466 0" xyz="0.555975 0 0.72404" />
+    <parent link="base_link" />
+    <child link="camera_link" />
   </joint>
   <link name="imu_link">
     <visual>
-      <origin rpy="0 0 0" xyz="0 0 0"/>
-      <geometry>
-        <box size="0.05 0.05 0.05"/>
-      </geometry>
-      <material name="Blue"/>
+      <origin rpy="0 0 0" xyz="0 0 0" />
+      <geometry>
+        <box size="0.05 0.05 0.05" />
+      </geometry>
+      <material name="Blue" />
     </visual>
   </link>
   <joint name="imu_joint" type="fixed">
-    <origin rpy="0 0 0" xyz="0.16 0 0"/>
-    <parent link="base_link"/>
-    <child link="imu_link"/>
+    <origin rpy="0 0 0" xyz="0.16 0 0" />
+    <parent link="base_link" />
+    <child link="imu_link" />
   </joint>
   <link name="gps_link">
     <visual>
-      <origin rpy="0 0 0" xyz="0 0 0"/>
-      <geometry>
-        <box size="0.1 0.1 0.1"/>
-      </geometry>
-      <material name="Blue"/>
+      <origin rpy="0 0 0" xyz="0 0 0" />
+      <geometry>
+        <box size="0.1 0.1 0.1" />
+      </geometry>
+      <material name="Blue" />
     </visual>
   </link>
   <joint name="gps_joint" type="fixed">
-    <origin rpy="0 0 0" xyz="0.16 0 0.48011"/>
-    <parent link="base_link"/>
-    <child link="gps_link"/>
+    <origin rpy="0 0 0" xyz="0.16 0 0.48011" />
+    <parent link="base_link" />
+    <child link="gps_link" />
   </joint>
   <gazebo>
     <plugin name="differential_drive_controller" filename="libgazebo_ros_diff_drive.so">
       <leftJoint>left_wheel_joint</leftJoint>
+      <odometryTopic>odom</odometryTopic>
+      <odometryFrame>odom</odometryFrame>
+      <publishWheelTF>false</publishWheelTF>
+      <publishOdomTF>true</publishOdomTF>
+      <wheelTorque>5</wheelTorque>
+      <wheelAcceleration>0</wheelAcceleration>
+      <updateRate>100</updateRate>
+      <odometrySource>world</odometrySource> <!-- 'encoder' instead of 'world' is also possible -->
+      <publishTf>1</publishTf>
+      <rosDebugLevel>na</rosDebugLevel>
       <rightJoint>right_wheel_joint</rightJoint>
       <robotBaseFrame>base_link</robotBaseFrame>
@@ -242,5 +252,5 @@
       <pose>0 0 0 0 0 0</pose>
       <visualize>true</visualize>
-      <update_rate>25</update_rate>      <!-- choosen for SICK LMS111-->
+      <update_rate>25</update_rate> <!-- choosen for SICK LMS111-->
       <ray>
         <scan>
@@ -264,5 +274,5 @@
     </sensor>
   </gazebo>
-<gazebo reference="camera_link">
+  <gazebo reference="camera_link">
     <sensor type="camera" name="camera1">
       <update_rate>30.0</update_rate>
